Commit message: running object robot, todo: params as launch params

File: rrbot_description/urdf/rrbot.xacro (robot description, xacro)
@@ -4,11 +4,11 @@
   <!-- Constants for robot dimensions -->
   <xacro:property name="PI" value="3.1415926535897931"/>
-  <xacro:property name="mass" value="1" /> <!-- arbitrary value for mass -->
-  <xacro:property name="width" value="0.1" /> <!-- Square dimensions (widthxwidth) of beams -->
-  <xacro:property name="height1" value="2" /> <!-- Link 1 -->
-  <xacro:property name="height2" value="1" /> <!-- Link 2 -->
-  <xacro:property name="height3" value="1" /> <!-- Link 3 -->
-  <xacro:property name="camera_link" value="0.05" /> <!-- Size of square 'camera' box -->
-  <xacro:property name="axel_offset" value="0.05" /> <!-- Space btw top of beam and the each joint -->
+  <xacro:property name="mass" value="1" />
+  <xacro:property name="pos_x" value="2" />
+  <xacro:property name="pos_y" value="0" />
+  <xacro:property name="pos_z" value="1" />
+  <xacro:property name="obj_x" value="0.25" />
+  <xacro:property name="obj_y" value="0.25" />
+  <xacro:property name="obj_z" value="0.25" />
   <!-- Import all Gazebo-customization elements, including Gazebo colors -->
   <xacro:include filename="$(find rrbot_description)/urdf/rrbot.gazebo" />
@@ -54,9 +54,27 @@
     <child link="link3"/>
     <origin xyz="0 0 0" rpy="0 0 0"/>
-    <axis xyz="0 0 -1"/>
+    <axis xyz="0 0 1"/>
+    <dynamics damping="0.3"/>
+  </joint>
+  <!-- Middle Link -->
+  <link name="link3">
+    <inertial>
+      <origin xyz="0 0 0.01" rpy="0 0 0"/>
+      <mass value="${mass}"/>
+      <inertia
+      ixx="0.0" ixy="0.0" ixz="0.0"
+	  iyy="0.0" iyz="0.0"
+	  izz="0.0"/>
+    </inertial>
+  </link>
+  <joint name="joint3" type="continuous">
+    <parent link="link3"/>
+    <child link="link4"/>
+    <origin xyz="${pos_x} ${pos_y} ${pos_z}" rpy="0 0 0"/>
+    <axis xyz="1 0 0"/>
     <dynamics damping="0.3"/>
   </joint>
   <!-- Top Link -->
-  <link name="link3">
+  <link name="link4">
     <inertial>
       <origin xyz="0 0 0.1" rpy="0 0 0"/>
@@ -67,12 +85,19 @@
 	  izz="0.0"/>
     </inertial>
+    <visual>
+      <origin xyz="0 0 0" rpy="0 0 0"/>
+      <geometry>
+        <box size="${obj_x} ${obj_y} ${obj_z}"/>
+      </geometry>
+      <material name="gray"/>
+    </visual>
   </link>
   <transmission name="tran1">
     <type>transmission_interface/SimpleTransmission</type>
     <joint name="joint1">
-      <hardwareInterface>hardware_interface/EffortJointInterface</hardwareInterface>
+      <hardwareInterface>hardware_interface/VelocityJointInterface</hardwareInterface>
     </joint>
     <actuator name="motor1">
-      <hardwareInterface>hardware_interface/EffortJointInterface</hardwareInterface>
+      <hardwareInterface>hardware_interface/VelocityJointInterface</hardwareInterface>
       <mechanicalReduction>1</mechanicalReduction>
     </actuator>
@@ -81,8 +106,18 @@
     <type>transmission_interface/SimpleTransmission</type>
     <joint name="joint2">
-      <hardwareInterface>hardware_interface/EffortJointInterface</hardwareInterface>
+      <hardwareInterface>hardware_interface/VelocityJointInterface</hardwareInterface>
     </joint>
     <actuator name="motor2">
-      <hardwareInterface>hardware_interface/EffortJointInterface</hardwareInterface>
+      <hardwareInterface>hardware_interface/VelocityJointInterface</hardwareInterface>
+      <mechanicalReduction>1</mechanicalReduction>
+    </actuator>
+  </transmission>
+  <transmission name="tran3">
+    <type>transmission_interface/SimpleTransmission</type>
+    <joint name="joint3">
+      <hardwareInterface>hardware_interface/VelocityJointInterface</hardwareInterface>
+    </joint>
+    <actuator name="motor3">
+      <hardwareInterface>hardware_interface/VelocityJointInterface</hardwareInterface>
       <mechanicalReduction>1</mechanicalReduction>
     </actuator>
