Commit message: savme stick as actor

File: rrbot_description/urdf/my_actor.urdf.xacro (robot description, xacro)
@@ -8,6 +8,6 @@
   <xacro:my_actor.actor parent="$(arg parent)" ns="$(arg ns)">
     <origin xyz="0 0 0" rpy="0 0 0" />
-    <origin xyz="1 0 0" rpy="0 0 0" />
-    <box size="0.1 0.1 0.1" />
+    <origin xyz="2 -0.095 0.055" rpy="0 0 0" />
+    <box size="0.1 0.1 5.5" />
   </xacro:my_actor.actor>
 </robot>
