Commit message: colors and stuff for validation ring tests

File: rrbot_description/urdf/actor.gazebo.xacro (robot description, xacro)
@@ -7,4 +7,13 @@
       </plugin>
     </gazebo>
+    <gazebo reference="${prefix}link_2">
+      <material>Gazebo/LightGrey</material>
+    </gazebo>
+    <gazebo reference="${prefix}link_separate_mesh">
+      <material>Gazebo/LightGrey</material>
+    </gazebo>
+    <gazebo reference="${prefix}link_3">
+      <material>Gazebo/Blue</material>
+    </gazebo>
   </xacro:macro>
 </robot>

File: rrbot_description/urdf/actor.urdf.xacro (robot description, xacro)
@@ -15,5 +15,4 @@
     <xacro:include filename="$(find rrbot_description)/urdf/actor.gazebo.xacro" />
     <xacro:include filename="$(find rrbot_description)/urdf/materials.urdf.xacro" />
-    <xacro:actor_materials />
     <joint name="${prefix}base_joint" type="fixed">
       <xacro:insert_block name="actor_origin" />
@@ -36,5 +35,4 @@
       <origin xyz="0 0 0" rpy="0 0 0"/>
       <axis xyz="0 1 0"/>
-      <dynamics damping="0.3"/>
     </joint>
     <link name="${prefix}link_1">
@@ -53,5 +51,4 @@
       <origin xyz="0 0 0" rpy="0 0 0"/>
       <axis xyz="0 0 1"/>
-      <dynamics damping="0.3"/>
     </joint>
     <!-- Middle Link -->
@@ -65,4 +62,25 @@
   	    izz="0.0"/>
       </inertial>
+      <visual>
+        <origin xyz="0 -0.05 0" rpy="${PI/2} 0 0"/>
+        <geometry>
+          <mesh filename="package://rrbot_description/meshes/validation_ring_v3.stl" scale="1 1 1"/>
+        </geometry>
+        <material name="black" />
+      </visual>
+    </link>
+    <joint name="${prefix}add_2nd_mesh" type="fixed">
+      <parent link="${prefix}link_2"/>
+      <child link="${prefix}link_separate_mesh"/>
+    </joint>
+    <!-- Middle Link -->
+    <link name="${prefix}link_separate_mesh">
+      <visual>
+        <origin xyz="0 0.05 0" rpy="${PI/2} 0 ${PI}"/>
+        <geometry>
+          <mesh filename="package://rrbot_description/meshes/validation_ring_v3.stl" scale="1 1 1"/>
+        </geometry>
+        <material name="white" />
+      </visual>
     </link>
     <joint name="${prefix}joint_3" type="continuous">
@@ -84,11 +102,4 @@
   	    izz="0.0"/>
       </inertial>
-      <visual>
-        <origin xyz="0 0 0" rpy="0 0 0"/>
-        <geometry>
-          <xacro:insert_block name="obj_shape" />
-        </geometry>
-        <material name="grey"/>
-      </visual>
     </link>
     <xacro:actor_transmission prefix="${ns}_" />

File: rrbot_description/urdf/materials.urdf.xacro (robot description, xacro)
@@ -1,5 +1,4 @@
 <?xml version="1.0"?>
 <robot xmlns:xacro="http://www.ros.org/wiki/xacro">
-  <xacro:macro name="actor_materials">
     <material name="black">
       <color rgba="0.0 0.0 0.0 1.0"/>
@@ -26,4 +25,3 @@
       <color rgba="1.0 1.0 1.0 1.0"/>
     </material>
-  </xacro:macro>
 </robot>

File: rrbot_description/urdf/my_actor.urdf.xacro (robot description, xacro)
@@ -7,5 +7,5 @@
   </link>
   <xacro:my_actor.actor parent="$(arg parent)" ns="$(arg ns)">
-    <origin xyz="0 0 0" rpy="0 0 0" />
+    <origin xyz="0 -0.095 0.055" rpy="0 0 0" />
     <origin xyz="2 -0.095 0.055" rpy="0 0 0" />
     <box size="0.1 0.1 5.5" />

Commit message: experiment v1 status!

File: rrbot_description/urdf/actor.gazebo.xacro (robot description, xacro)
@@ -14,5 +14,5 @@
     </gazebo>
     <gazebo reference="${prefix}link_3">
-      <material>Gazebo/Blue</material>
+      <material>Gazebo/Grey</material>
     </gazebo>
   </xacro:macro>

File: rrbot_description/urdf/actor.urdf.xacro (robot description, xacro)
@@ -62,11 +62,4 @@
   	    izz="0.0"/>
       </inertial>
-      <visual>
-        <origin xyz="0 0 0" rpy="0 0 0"/>
-        <geometry>
-          <mesh filename="package://rrbot_description/meshes/spherical_ring.stl" scale="2 2 2"/>
-        </geometry>
-        <material name="black" />
-      </visual>
     </link>
     <joint name="${prefix}joint_3" type="continuous">
@@ -88,4 +81,10 @@
   	    izz="0.0"/>
       </inertial>
+      <visual>
+        <geometry>
+          <xacro:insert_block name="obj_shape" />
+        </geometry>
+        <material name="black" />
+      </visual>
     </link>
     <xacro:actor_transmission prefix="${ns}_" />
@@ -93,3 +92,2 @@
   </xacro:macro>
 </robot>
-          <!--<box size="${obj_x} ${obj_y} ${obj_z}"/>-->

File: rrbot_description/urdf/my_actor.urdf.xacro (robot description, xacro)
@@ -8,6 +8,6 @@
   <xacro:my_actor.actor parent="$(arg parent)" ns="$(arg ns)">
     <origin xyz="0 -0.095 0.055" rpy="0 0 0" />
-    <origin xyz="2 0.0 0.0" rpy="0 0 0" />
-    <box size="0.1 0.1 5.5" />
+    <origin xyz="1 0.0 0.0" rpy="0 0 0" />
+    <box size="0.5 0.5 0.5" />
   </xacro:my_actor.actor>
 </robot>
