Commit message: coordinates/translations adjusted

File: rrbot_description/urdf/actor.urdf.xacro (robot description, xacro)
@@ -63,23 +63,9 @@
       </inertial>
       <visual>
-        <origin xyz="0 -0.05 0" rpy="${PI/2} 0 0"/>
+        <origin xyz="0 0 0" rpy="0 0 0"/>
         <geometry>
-          <mesh filename="package://rrbot_description/meshes/validation_ring_v3.stl" scale="1 1 1"/>
+          <mesh filename="package://rrbot_description/meshes/spherical_ring.stl" scale="2 2 2"/>
         </geometry>
         <material name="black" />
-      </visual>
-    </link>
-    <joint name="${prefix}add_2nd_mesh" type="fixed">
-      <parent link="${prefix}link_2"/>
-      <child link="${prefix}link_separate_mesh"/>
-    </joint>
-    <!-- Middle Link -->
-    <link name="${prefix}link_separate_mesh">
-      <visual>
-        <origin xyz="0 0.05 0" rpy="${PI/2} 0 ${PI}"/>
-        <geometry>
-          <mesh filename="package://rrbot_description/meshes/validation_ring_v3.stl" scale="1 1 1"/>
-        </geometry>
-        <material name="white" />
       </visual>
     </link>

File: rrbot_description/urdf/my_actor.urdf.xacro (robot description, xacro)
@@ -8,5 +8,5 @@
   <xacro:my_actor.actor parent="$(arg parent)" ns="$(arg ns)">
     <origin xyz="0 -0.095 0.055" rpy="0 0 0" />
-    <origin xyz="2 -0.095 0.055" rpy="0 0 0" />
+    <origin xyz="2 0.0 0.0" rpy="0 0 0" />
     <box size="0.1 0.1 5.5" />
   </xacro:my_actor.actor>

Commit message: settings for vali_1

File: rrbot_description/urdf/actor.urdf.xacro (robot description, xacro)
@@ -82,6 +82,7 @@
       </inertial>
       <visual>
+        <origin xyz="0 0 0" rpy="0 -${pi/2} 0"/>
         <geometry>
-          <xacro:insert_block name="obj_shape" />
+          <mesh filename="package://rrbot_description/meshes/spherical_ring.stl" scale="2 2 2"/>
         </geometry>
         <material name="black" />

File: rrbot_description/urdf/my_actor.urdf.xacro (robot description, xacro)
@@ -8,5 +8,5 @@
   <xacro:my_actor.actor parent="$(arg parent)" ns="$(arg ns)">
     <origin xyz="0 -0.095 0.055" rpy="0 0 0" />
-    <origin xyz="1 0.0 0.0" rpy="0 0 0" />
+    <origin xyz="0.0 0.0 0.0" rpy="0 0 0" />
     <box size="0.5 0.5 0.5" />
   </xacro:my_actor.actor>
